File: beacon-pcb/beacon-pcb.kicad_pcb (KiCad board)
At the start: 2 copper layers, 113.5 x 16.5 mm, 7 parts, among them IC1 BT832, J1 TC2030-CTX-NL

Commit message: Release beacon PCB for manufacture.
Parts:
- removed sticker: sticker, sticker
- added C2: 15p, Capacitor_SMD:C_0603_1608Metric_Pad1.05x0.95mm_HandSolder, F.Cu at (173.8, 110.2)
- added C3: 15p, Capacitor_SMD:C_0603_1608Metric_Pad1.05x0.95mm_HandSolder, F.Cu at (173.8, 117.2)
- added Y1: 32.768kHz, Crystal:Crystal_SMD_3215-2Pin_3.2x1.5mm, F.Cu at (173.8, 113.8)
- added dcfurs-logo: dcfurs-logo, dcfurs-logo, F.Cu at (109.2, 111.8)
Routing:
- net GND: track 23.1 -> 51.4 mm, vias 1 -> 3
- net Net-(C2-Pad1): track 0.00 -> 6.19 mm
- net Net-(C3-Pad1): track 0.00 -> 6.14 mm
Other:
- board text added: "DCFurs Bluetooth Beacon This device complies with part 15 of the Furry Communications Commission Rules. Operation is subject to the following two conditions: (1) This device may not cause harmful awoos, and (2) this device must accept any hugs and scritches, including those that may cause undesired attention."
- board text removed: "DCFurs Bluetooth Beacon This device complies with part 15 of the Furry Communications Commission Rules. Operation is subject to the following two conditions: (1) This device may not cause harmful awoos, and (2) this device must accept any hugs and scritches, including those that may cause undesired affection. Art: Nowandlater"
